File: keypad/keypad.brd (EAGLE design)
At the start: 34.3 x 40.1 mm, 16 parts, among them U1 SX1509

Commit message: added in changes to the lcd to use 4 wire interface updated other schematics to have cascading of interrupt
Parts:
- removed R4: 10k, SparkFun-Passives:0402-RES
Connections:
- removed net 13: U1.21
- removed net 15: U1.22
- removed net NINT: R4.1, U1.9
- new net EXTERNAL_INTERRUPT: I2CIN.2, U1.22
- new net INTERNAL_INTERRUPT: I2COUT.2, U1.21, U1.9
- net 3.3V: no longer R4.2
- net GND: no longer I2CIN.2, I2COUT.2
Routing:
- net GND: track 91.7 -> 68.6 mm
- net NINT: track 4.92 -> 0.00 mm
Changed lines of the file:
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@@
 <element name="R2" library="SparkFun-Passives" package="0402-RES" value="10k" x="5.08" y="73.66" rot="R180"/>
 <element name="R3" library="SparkFun-Passives" package="0402-RES" value="10k" x="3.81" y="76.2" rot="R180"/>
-<element name="R4" library="SparkFun-Passives" package="0402-RES" value="10k" x="16.51" y="65.278" rot="R270"/>
 <element name="SJ3" library="SparkFun-Passives" package="SJ_2S-NO" value="" x="3.81" y="67.31" rot="R90"/>
 <element name="SJ4" library="SparkFun-Passives" package="SJ_2S-NO" value="" x="7.62" y="63.5" rot="R180"/>
@@
 <contactref element="U1" pad="17"/>
 <contactref element="U1" pad="29"/>
-<contactref element="I2CIN" pad="2"/>
 <contactref element="I2CIN" pad="1"/>
-<contactref element="I2COUT" pad="2"/>
 <contactref element="I2COUT" pad="1"/>
 <contactref element="S1" pad="1"/>
 <contactref element="S2" pad="1"/>
-<wire x1="30.099" y1="84.074" x2="28.829" y2="82.804" width="0.254" layer="1"/>
 <wire x1="30.099" y1="85.344" x2="30.099" y2="84.074" width="0.254" layer="1"/>
-<wire x1="13.335" y1="84.074" x2="12.065" y2="82.804" width="0.254" layer="1"/>
 <wire x1="13.335" y1="85.344" x2="13.335" y2="84.074" width="0.254" layer="1"/>
 <wire x1="9.652" y1="65.913" x2="7.62" y2="67.945" width="0.254" layer="1"/>
@@
 <wire x1="11.43" y1="61.595" x2="11.43" y2="61.58" width="0.254" layer="1"/>
 <wire x1="10.033" y1="80.772" x2="10.8585" y2="81.5975" width="0.254" layer="1"/>
-<wire x1="10.8585" y1="81.5975" x2="12.065" y2="82.804" width="0.254" layer="1"/>
 <wire x1="10.033" y1="70.485" x2="10.033" y2="80.772" width="0.254" layer="1"/>
 <wire x1="7.62" y1="68.072" x2="10.033" y2="70.485" width="0.254" layer="1"/>
 <wire x1="7.62" y1="68.072" x2="7.62" y2="67.96" width="0.254" layer="1"/>
-<wire x1="27.559" y1="81.534" x2="28.829" y2="82.804" width="0.254" layer="1"/>
 <wire x1="10.922" y1="81.534" x2="10.8585" y2="81.5975" width="0.254" layer="1"/>
 <wire x1="18.345" y1="71.52" x2="11.068" y2="71.52" width="0.254" layer="1"/>
@@
 <wire x1="22.8346" y1="60.1726" x2="22.824" y2="60.17" width="0.254" layer="1"/>
 <wire x1="13.1318" y1="61.5696" x2="13.0556" y2="61.6712" width="0.254" layer="1"/>
-<wire x1="27.559" y1="81.534" x2="13.462" y2="81.534" width="0.254" layer="1"/>
-<wire x1="13.462" y1="81.534" x2="12.065" y2="82.804" width="0.254" layer="1"/>
+<wire x1="22.295" y1="70.72" x2="30.099" y2="84.074" width="0" layer="19" extent="1-1"/>
+<wire x1="13.335" y1="84.074" x2="10.922" y2="81.534" width="0" layer="19" extent="1-1"/>
 </signal>
 <signal name="3.3V">
@@
 <contactref element="U1" pad="12"/>
 <contactref element="R1" pad="2"/>
-<contactref element="R4" pad="2"/>
 <contactref element="SJ4" pad="2"/>
 <contactref element="SJ3" pad="2"/>
@@
 <via x="7.9756" y="62.1538" extent="1-16" drill="0.6096"/>
 <wire x1="14.8336" y1="64.643" x2="16.51" y2="64.643" width="0.254" layer="1"/>
-<wire x1="16.51" y1="64.643" x2="16.51" y2="64.628" width="0.254" layer="1"/>
 <wire x1="14.8336" y1="64.643" x2="14.732" y2="64.658" width="0.254" layer="1"/>
 <wire x1="18.3134" y1="62.7634" x2="16.5608" y2="64.516" width="0.254" layer="1"/>
 <wire x1="18.3134" y1="60.1726" x2="18.3134" y2="62.7634" width="0.254" layer="1"/>
-<wire x1="16.5608" y1="64.516" x2="16.51" y2="64.628" width="0.254" layer="1"/>
 <wire x1="18.3134" y1="60.1726" x2="18.324" y2="60.17" width="0.254" layer="1"/>
 <wire x1="20.72" y1="69.145" x2="20.574" y2="67.818" width="0.254" layer="1"/>
 <wire x1="20.574" y1="67.818" x2="20.574" y2="64.77" width="0.254" layer="1"/>
 <wire x1="20.574" y1="64.77" x2="16.764" y2="64.77" width="0.254" layer="1"/>
-<wire x1="16.764" y1="64.77" x2="16.51" y2="64.628" width="0.254" layer="1"/>
+<wire x1="16.51" y1="64.643" x2="16.764" y2="64.77" width="0" layer="19" extent="1-1"/>
+<wire x1="16.5608" y1="64.516" x2="16.51" y2="64.643" width="0" layer="19" extent="1-1"/>
 </signal>
 <signal name="14">
 <contactref element="U1" pad="20"/>
-</signal>
-<signal name="15">
-<contactref element="U1" pad="22"/>
 </signal>
 <signal name="ROW_1-3">
@@
 <wire x1="19.558" y1="77.47" x2="7.62" y2="77.47" width="0.254" layer="16"/>
 </signal>
-<signal name="NINT">
-<contactref element="U1" pad="9"/>
-<contactref element="R4" pad="1"/>
-<wire x1="19.52" y1="69.145" x2="19.05" y2="67.056" width="0.254" layer="1"/>
-<wire x1="19.05" y1="67.056" x2="16.51" y2="65.928" width="0.254" layer="1"/>
-</signal>
 <signal name="OSCIO">
 <contactref element="U1" pad="11"/>
@@
 <wire x1="19.12" y1="73.095" x2="18.288" y2="73.787" width="0.254" layer="1"/>
 </signal>
-<signal name="13">
-<contactref element="U1" pad="21"/>
-</signal>
 <signal name="8">
 <contactref element="U1" pad="7"/>
@@
 <wire x1="22.352" y1="69.85" x2="22.295" y2="69.92" width="0.254" layer="1"/>
 </signal>
+<signal name="EXTERNAL_INTERRUPT">
+<contactref element="I2CIN" pad="2"/>
+<contactref element="U1" pad="22"/>
+<wire x1="21.52" y1="73.095" x2="28.829" y2="82.804" width="0" layer="19" extent="1-1"/>
+</signal>
+<signal name="INTERNAL_INTERRUPT">
+<contactref element="I2COUT" pad="2"/>
+<contactref element="U1" pad="9"/>
+<contactref element="U1" pad="21"/>
+<wire x1="22.295" y1="72.32" x2="12.065" y2="82.804" width="0" layer="19" extent="1-1"/>
+<wire x1="19.52" y1="69.145" x2="22.295" y2="72.32" width="0" layer="19" extent="1-1"/>
+</signal>
 </signals>
