File: keypad/keypad.sch (EAGLE design)
At the start: 16 parts, among them U1 SX1509

Commit message: added in changes to the lcd to use 4 wire interface updated other schematics to have cascading of interrupt
Parts:
- removed R4: 10k, SparkFun-Passives:RESISTOR0402-RES
Connections:
- removed net 13: U1.I/O[14]
- removed net 15: U1.I/O[15]
- removed net NINT: R4.1, U1.!INT
- new net EXTERNAL_INTERRUPT: I2CIN.2, U1.I/O[15]
- new net INTERNAL_INTERRUPT: I2COUT.2, U1.!INT, U1.I/O[14]
- net 3.3V: no longer R4.2
- net GND: no longer I2CIN.2, I2COUT.2
Changed lines of the file:
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@@
 <part name="R2" library="SparkFun-Passives" deviceset="RESISTOR" device="0402-RES" value="10k"/>
 <part name="R3" library="SparkFun-Passives" deviceset="RESISTOR" device="0402-RES" value="10k"/>
-<part name="R4" library="SparkFun-Passives" deviceset="RESISTOR" device="0402-RES" value="10k"/>
 <part name="P+2" library="SparkFun-Aesthetics" deviceset="3.3V" device=""/>
 <part name="GND4" library="SparkFun-Aesthetics" deviceset="GND" device=""/>
@@
 <attribute name="VALUE" x="56.642" y="67.31" size="1.778" layer="96" rot="R90"/>
 </instance>
-<instance part="R4" gate="G$1" x="76.2" y="66.04" smashed="yes" rot="R90">
-<attribute name="NAME" x="79.5274" y="62.23" size="1.778" layer="95" rot="R90"/>
-<attribute name="VALUE" x="79.502" y="67.31" size="1.778" layer="96" rot="R90"/>
-</instance>
 <instance part="P+2" gate="G$1" x="81.28" y="81.28"/>
 <instance part="GND4" gate="1" x="91.44" y="22.86"/>
@@
 </segment>
 <segment>
-<pinref part="I2CIN" gate="G$1" pin="2"/>
 <pinref part="I2CIN" gate="G$1" pin="1"/>
-<wire x1="12.7" y1="53.34" x2="12.7" y2="50.8" width="0.1524" layer="91"/>
 <pinref part="GND6" gate="1" pin="GND"/>
 <wire x1="12.7" y1="50.8" x2="17.78" y2="50.8" width="0.1524" layer="91"/>
 <wire x1="17.78" y1="50.8" x2="17.78" y2="43.18" width="0.1524" layer="91"/>
-<junction x="12.7" y="50.8"/>
-</segment>
-<segment>
-<pinref part="I2COUT" gate="G$1" pin="2"/>
+</segment>
+<segment>
 <pinref part="I2COUT" gate="G$1" pin="1"/>
-<wire x1="10.16" y1="17.78" x2="10.16" y2="15.24" width="0.1524" layer="91"/>
 <pinref part="GND9" gate="1" pin="GND"/>
 <wire x1="10.16" y1="15.24" x2="12.7" y2="15.24" width="0.1524" layer="91"/>
 <wire x1="12.7" y1="15.24" x2="12.7" y2="10.16" width="0.1524" layer="91"/>
-<junction x="10.16" y="15.24"/>
 </segment>
 <segment>
@@
 <wire x1="81.28" y1="73.66" x2="81.28" y2="71.12" width="0.1524" layer="91"/>
 <junction x="81.28" y="73.66"/>
-<pinref part="R4" gate="G$1" pin="2"/>
-<wire x1="76.2" y1="71.12" x2="76.2" y2="73.66" width="0.1524" layer="91"/>
-<wire x1="76.2" y1="73.66" x2="81.28" y2="73.66" width="0.1524" layer="91"/>
 </segment>
 <segment>
@@
 <wire x1="119.38" y1="33.02" x2="121.92" y2="33.02" width="0.1524" layer="91"/>
 <label x="121.92" y="33.02" size="1.27" layer="95" xref="yes"/>
-</segment>
-</net>
-<net name="15" class="0">
-<segment>
-<pinref part="U1" gate="G$1" pin="I/O[15]"/>
-<wire x1="119.38" y1="27.94" x2="121.92" y2="27.94" width="0.1524" layer="91"/>
-<label x="121.92" y="27.94" size="1.27" layer="95" xref="yes"/>
 </segment>
 </net>
@@
 </segment>
 <segment>
-<label x="17.78" y="55.88" size="1.778" layer="95" xref="yes"/>
+<label x="15.24" y="60.96" size="1.778" layer="95" xref="yes"/>
 <pinref part="I2CIN" gate="G$1" pin="5"/>
-<wire x1="17.78" y1="55.88" x2="12.7" y2="60.96" width="0.1524" layer="91"/>
+<wire x1="15.24" y1="60.96" x2="12.7" y2="60.96" width="0.1524" layer="91"/>
 <pinref part="I2CIN" gate="G$1" pin="4"/>
 <wire x1="12.7" y1="58.42" x2="12.7" y2="60.96" width="0.1524" layer="91"/>
@@
 </segment>
 <segment>
-<label x="15.24" y="20.32" size="1.778" layer="95" xref="yes"/>
+<label x="12.7" y="25.4" size="1.778" layer="95" xref="yes"/>
 <pinref part="I2COUT" gate="G$1" pin="5"/>
-<wire x1="10.16" y1="25.4" x2="15.24" y2="20.32" width="0.1524" layer="91"/>
+<wire x1="10.16" y1="25.4" x2="12.7" y2="25.4" width="0.1524" layer="91"/>
 <pinref part="I2COUT" gate="G$1" pin="4"/>
 <wire x1="10.16" y1="25.4" x2="10.16" y2="22.86" width="0.1524" layer="91"/>
@@
 <segment>
 <pinref part="I2CIN" gate="G$1" pin="6"/>
-<wire x1="17.78" y1="63.5" x2="12.7" y2="63.5" width="0.1524" layer="91"/>
-<label x="17.78" y="63.5" size="1.778" layer="95" xref="yes"/>
+<wire x1="25.4" y1="63.5" x2="12.7" y2="63.5" width="0.1524" layer="91"/>
+<label x="25.4" y="63.5" size="1.778" layer="95" xref="yes"/>
 <pinref part="I2CIN" gate="G$1" pin="3"/>
-<wire x1="17.78" y1="63.5" x2="17.78" y2="60.96" width="0.1524" layer="91"/>
-<wire x1="17.78" y1="60.96" x2="12.7" y2="55.88" width="0.1524" layer="91"/>
+<wire x1="25.4" y1="63.5" x2="25.4" y2="55.88" width="0.1524" layer="91"/>
+<wire x1="25.4" y1="55.88" x2="12.7" y2="55.88" width="0.1524" layer="91"/>
 </segment>
 <segment>
 <pinref part="I2COUT" gate="G$1" pin="6"/>
-<wire x1="12.7" y1="27.94" x2="10.16" y2="27.94" width="0.1524" layer="91"/>
-<label x="12.7" y="27.94" size="1.778" layer="95" xref="yes"/>
+<wire x1="22.86" y1="27.94" x2="10.16" y2="27.94" width="0.1524" layer="91"/>
+<label x="22.86" y="27.94" size="1.778" layer="95" xref="yes"/>
 <pinref part="I2COUT" gate="G$1" pin="3"/>
-<wire x1="12.7" y1="27.94" x2="12.7" y2="22.86" width="0.1524" layer="91"/>
-<wire x1="12.7" y1="22.86" x2="10.16" y2="20.32" width="0.1524" layer="91"/>
-</segment>
-</net>
-<net name="NINT" class="0">
-<segment>
-<pinref part="U1" gate="G$1" pin="!INT"/>
-<pinref part="R4" gate="G$1" pin="1"/>
-<wire x1="93.98" y1="45.72" x2="76.2" y2="45.72" width="0.1524" layer="91"/>
-<wire x1="76.2" y1="45.72" x2="76.2" y2="60.96" width="0.1524" layer="91"/>
-<label x="91.44" y="45.72" size="1.778" layer="95" rot="MR0"/>
+<wire x1="22.86" y1="27.94" x2="22.86" y2="20.32" width="0.1524" layer="91"/>
+<wire x1="22.86" y1="20.32" x2="10.16" y2="20.32" width="0.1524" layer="91"/>
 </segment>
 </net>
@@
 </segment>
 </net>
-<net name="13" class="0">
+<net name="8" class="0">
+<segment>
+<pinref part="U1" gate="G$1" pin="I/O[6]"/>
+<wire x1="119.38" y1="55.88" x2="121.92" y2="55.88" width="0.1524" layer="91"/>
+<label x="121.92" y="55.88" size="1.27" layer="95" xref="yes"/>
+</segment>
+</net>
+<net name="9" class="0">
+<segment>
+<pinref part="U1" gate="G$1" pin="I/O[5]"/>
+<wire x1="119.38" y1="58.42" x2="121.92" y2="58.42" width="0.1524" layer="91"/>
+<label x="121.92" y="58.42" size="1.27" layer="95" xref="yes"/>
+</segment>
+</net>
+<net name="10" class="0">
+<segment>
+<pinref part="U1" gate="G$1" pin="I/O[4]"/>
+<wire x1="119.38" y1="60.96" x2="121.92" y2="60.96" width="0.1524" layer="91"/>
+<label x="121.92" y="60.96" size="1.27" layer="95" xref="yes"/>
+</segment>
+</net>
+<net name="ROW_STAR-POUND" class="0">
+<segment>
+<pinref part="U1" gate="G$1" pin="I/O[3]"/>
+<wire x1="119.38" y1="63.5" x2="121.92" y2="63.5" width="0.1524" layer="91"/>
+<label x="121.92" y="63.5" size="1.27" layer="95" xref="yes"/>
+</segment>
+</net>
+<net name="ROW_7-9" class="0">
+<segment>
+<pinref part="U1" gate="G$1" pin="I/O[2]"/>
+<wire x1="119.38" y1="66.04" x2="121.92" y2="66.04" width="0.1524" layer="91"/>
+<label x="121.92" y="66.04" size="1.27" layer="95" xref="yes"/>
+</segment>
+</net>
+<net name="EXTERNAL_INTERRUPT" class="0">
+<segment>
+<pinref part="I2CIN" gate="G$1" pin="2"/>
+<wire x1="12.7" y1="53.34" x2="17.78" y2="53.34" width="0.1524" layer="91"/>
+<label x="17.78" y="53.34" size="1.778" layer="95" xref="yes"/>
+</segment>
+<segment>
+<pinref part="U1" gate="G$1" pin="I/O[15]"/>
+<wire x1="119.38" y1="27.94" x2="121.92" y2="27.94" width="0.1524" layer="91"/>
+<label x="121.92" y="27.94" size="1.27" layer="95" xref="yes"/>
+</segment>
+</net>
+<net name="INTERNAL_INTERRUPT" class="0">
+<segment>
+<pinref part="I2COUT" gate="G$1" pin="2"/>
+<wire x1="10.16" y1="17.78" x2="12.7" y2="17.78" width="0.1524" layer="91"/>
+<label x="12.7" y="17.78" size="1.778" layer="95" xref="yes"/>
+</segment>
+<segment>
+<pinref part="U1" gate="G$1" pin="!INT"/>
+<wire x1="93.98" y1="45.72" x2="91.44" y2="45.72" width="0.1524" layer="91"/>
+<label x="91.44" y="45.72" size="1.778" layer="95" rot="R180" xref="yes"/>
+</segment>
 <segment>
 <pinref part="U1" gate="G$1" pin="I/O[14]"/>
@@
 </segment>
 </net>
-<net name="8" class="0">
-<segment>
-<pinref part="U1" gate="G$1" pin="I/O[6]"/>
-<wire x1="119.38" y1="55.88" x2="121.92" y2="55.88" width="0.1524" layer="91"/>
-<label x="121.92" y="55.88" size="1.27" layer="95" xref="yes"/>
-</segment>
-</net>
-<net name="9" class="0">
-<segment>
-<pinref part="U1" gate="G$1" pin="I/O[5]"/>
-<wire x1="119.38" y1="58.42" x2="121.92" y2="58.42" width="0.1524" layer="91"/>
-<label x="121.92" y="58.42" size="1.27" layer="95" xref="yes"/>
-</segment>
-</net>
-<net name="10" class="0">
-<segment>
-<pinref part="U1" gate="G$1" pin="I/O[4]"/>
-<wire x1="119.38" y1="60.96" x2="121.92" y2="60.96" width="0.1524" layer="91"/>
-<label x="121.92" y="60.96" size="1.27" layer="95" xref="yes"/>
-</segment>
-</net>
-<net name="ROW_STAR-POUND" class="0">
-<segment>
-<pinref part="U1" gate="G$1" pin="I/O[3]"/>
-<wire x1="119.38" y1="63.5" x2="121.92" y2="63.5" width="0.1524" layer="91"/>
-<label x="121.92" y="63.5" size="1.27" layer="95" xref="yes"/>
-</segment>
-</net>
-<net name="ROW_7-9" class="0">
-<segment>
-<pinref part="U1" gate="G$1" pin="I/O[2]"/>
-<wire x1="119.38" y1="66.04" x2="121.92" y2="66.04" width="0.1524" layer="91"/>
-<label x="121.92" y="66.04" size="1.27" layer="95" xref="yes"/>
-</segment>
-</net>
