File: lcd/LCD LED.sch (EAGLE design)
At the start: 23 parts, among them T1 MMDT3904, U1 SX1509

Commit message: added in changes to the lcd to use 4 wire interface updated other schematics to have cascading of interrupt
Parts:
- removed R4: 10k, SparkFun-Passives:RESISTOR0402-RES
- renumbered RV2 to CONTRAST
Connections:
- net VO renamed LCD_CONTRAST
- removed net 0: T_R7A.1, U1.I/O[1]
- removed net 1: T_R7B.1, U1.I/O[0]
- removed net 10: LCD1.DB5, U1.I/O[4]
- removed net 11: LCD1.DB6, U1.I/O[3]
- removed net 12: LCD1.DB7, U1.I/O[2]
- removed net 13: T_R7C.1, U1.I/O[14]
- removed net 14: T_R7D.1, U1.I/O[13]
- removed net 15: U1.I/O[15]
- removed net 2: LCD1.RS, U1.I/O[12]
- removed net 3: LCD1.R/W, U1.I/O[11]
- removed net 4: LCD1.E, U1.I/O[10]
- removed net 5: LCD1.DB0, U1.I/O[9]
- removed net 6: LCD1.DB1, U1.I/O[8]
- removed net 7: LCD1.DB2, U1.I/O[7]
- removed net 8: LCD1.DB3, U1.I/O[6]
- removed net 9: LCD1.DB4, U1.I/O[5]
- removed net NINT: R4.1, U1.!INT
- new net INTERRUPT_EXTERNAL: I2CIN.7, U1.I/O[15]
- new net INTERRUPT_INTERNAL: I2COUT.7, U1.!INT, U1.I/O[14]
- new net IO12: U1.I/O[12]
- new net IO13: U1.I/O[13]
- new net IO7: U1.I/O[7]
- new net LCD_BACKLIGHT: LCD1.A, U1.I/O[6]
- new net LCD_D0: LCD1.DB0
- new net LCD_D1: LCD1.DB1
- new net LCD_D2: LCD1.DB2
- new net LCD_D3: LCD1.DB3
- new net LCD_D4: LCD1.DB4, U1.I/O[2]
- new net LCD_D5: LCD1.DB5, U1.I/O[3]
- new net LCD_D6: LCD1.DB6, U1.I/O[4]
- new net LCD_D7: LCD1.DB7, U1.I/O[5]
- new net LCD_E: LCD1.E, U1.I/O[1]
- new net LCD_RS: LCD1.RS, U1.I/O[0]
- new net LED_1: T_R7A.1, U1.I/O[8]
- new net LED_2: T_R7B.1, U1.I/O[9]
- new net LED_3: T_R7C.1, U1.I/O[10]
- new net LED_4: T_R7D.1, U1.I/O[11]
- net 3.3V: now also C2.1, C3.1; no longer I2CIN.7, I2COUT.7, LCD1.A, R4.2
- net GND: now also LCD1.R/W
- net VCC1: no longer C3.1
- net VCC2: no longer C2.1
Other:
- moved on the sheet: C1, C2, C3, T1G$1, T1G$2, U$4G$2
